File: MicroController/Hardware/Distance sensors/Distance sensors.sch (EAGLE design)
At the start: 0 parts

Commit message: Added the necessary components for the Distance sensor shield.
Parts:
- added J1: (no value), SparkFun-Connectors:CONN_023.5MM
- added J10, J11, J12, J13, J14, J15, J16, J17, J2, J3, J4, J5, J6, J7, J8, J9: (no value), SparkFun-Connectors:CONN_04
- added U$1, U$2, U$3: RJ45-TRAFO, con-amphenol-rj45-ld:RJ45-TRAFO
