File: MicroController/Hardware/Control module/Control module.sch (EAGLE design)
At the start: 81 parts, among them CN1 JST-PH_2-PIN_HEADER, CN2 JST-PH_2-PIN_HEADER, CN3 JST-PH_2-PIN_HEADER, CN4 JST-PH_2-PIN_HEADER, CN5 JST-PH_2-PIN_HEADER, CN6 JST-PH_2-PIN_HEADER, CN7 JST-PH_2-PIN_HEADER, CN8 JST-PH_2-PIN_HEADER, IC1 MCP1703CB, J1 1X2-3.5MM, J2 RJ45-TRAFO, J3 RJ45-TRAFO, J4 RJ45-TRAFO, J6 RJ11, Q1 BSS138, Q2 BSS138, Q3 BSS138, Q4 BSS138, Q5 BSS138, Q6 BSS138, Q7 BSS138, Q8 BSS138, U1 CD74HC4067SM96, U3 TLV1117-33CDCY

Commit message: Major improvements
The Ultrasone PCB is in a good place now, it has also been well implemented on the control PCB.
Parts:
- removed C10: (no value), adafruit:CPOL-USE2.5-6
- removed C23, C24, C25: (no value), adafruit:C-USC0805
- added C4: (no value), adafruit:CPOL-US153CLV-0505
- added Q10, Q9: BSS138, SparkFun:MOSFET-NCHANNELSMD
- added R17, R18, R19, R20: 10K, SparkFun:RESISTOR0603-RES
- C5: device adafruit:CPOL-USE2.5-6 -> adafruit:CPOL-US153CLV-0505
Connections:
- new net ATXMEGA_TRIGGER_1: Q10.S, R19.2, U$1.PD2(OC0C/RXD0)
- new net ATXMEGA_TRIGGER_2: Q9.S, R17.2, U$1.PD1(OC0B/XCK0)
- net +12V: no longer C25.1, J2.GND
- net +5V: now also R18.1, R20.1; no longer C23.1, C24.1, J3.TX+, J4.TX+
- net A: now also U$1.PE7(TOSC1/CKOUT/EVO/TXD1/SCK)
- net B: now also U$1.PE6(TOSC2/RXD1/MISO)
- net C: now also U$1.PE5(OC1B/XCK1/MOSI)
- net GND: now also C4.-, J2.GND, J2.TX+, J3.TX+, J4.TX+; no longer C10.-, C23.2, C24.2, C25.2
- net S0: now also U$1.PC6(OC0DL/RXD1/MISO); no longer U$1.PD3(OX0D/TXD0)
- net S1: now also U$1.PC7(OC0DH/CKOUT/EVO/TXD1/SCK); no longer U$1.PD4(OC1A/SS)
- net S2: now also U$1.PC5(OC1B/OC0CH/XCK1/MOSI); no longer U$1.PD1(OC0B/XCK0)
- net S3: now also U$1.PC4(AC1A/OC0CL/SS); no longer U$1.PD0(OC0A)
- net TRIGGER_1: now also J4.RX0, Q10.D, R20.2; no longer J4.TX0, U$1.PB0(ADC0/AC0/AREF)
- net TRIGGER_2: now also J4.RX+, Q9.D, R18.2; no longer J4.TX-, U$1.PB1(ADC1/AC1)
- net ULTRA1: now also U1.CHAN3; no longer U1.CHAN0
- net ULTRA10: now also J4.TX0, U1.CHAN4; no longer J4.RX-, U1.CHAN9
- net ULTRA11: now also J3.NC1; no longer J4.RX0
- net ULTRA12: now also J3.RX-; no longer J4.RX+
- net ULTRA13: now also J3.RX0; no longer J3.TX0
- net ULTRA14: now also J3.RX+; no longer J3.TX-
- net ULTRA15: now also J3.TX-; no longer J3.RX+
- net ULTRA16: now also J3.TX0; no longer J3.RX0
- net ULTRA2: now also U1.CHAN2; no longer U1.CHAN1
- net ULTRA3: now also U1.CHAN1; no longer U1.CHAN2
- net ULTRA4: now also U1.CHAN0; no longer U1.CHAN3
- net ULTRA5: now also U1.CHAN8; no longer U1.CHAN4
- net ULTRA6: now also U1.CHAN9; no longer U1.CHAN5
- net ULTRA7: now also J4.NC1, U1.CHAN7; no longer J3.NC1, U1.CHAN6
- net ULTRA8: now also J4.RX-, U1.CHAN6; no longer J3.RX-, U1.CHAN7
- net ULTRA9: now also J4.TX-, U1.CHAN5; no longer J4.NC1, U1.CHAN8
- net ULTRA_COM: now also U$1.PD0(OC0A); no longer U$1.PD2(OC0C/RXD0)
- net VCC: now also C4.+, Q10.G, Q9.G, R17.1, R19.1; no longer C10.+

Commit message: Changed the Control PCB design to follow the Eurocircuits design rules.
Parts:
- removed C8: (no value), adafruit:C-USC0805
- added LED2: (no value), led:LEDCHIPLED_0805
- added R22: 10K, adafruit:R-US_R0805
- renumbered 12V_REGULATOR to U2, CN1 to MOTOR_1, CN2 to MOTOR_2, CN3 to MOTOR_3, CN4 to MOTOR_4, CN5 to MOTOR_5, CN6 to MOTOR_6, CN7 to MOTOR_7, CN8 to MOTOR_8, J5 to PDI_CONNECTOR
Connections:
- new net LED_1: R21.2, U$1.PD3(OX0D/TXD0)
- new net LED_2: R22.2, U$1.PD4(OC1A/SS)
- net +12V: no longer C8.1
- net GND: now also LED2.C; no longer C8.2
- net N$1: now also LED2.A, R22.1; no longer R21.2, U$1.PD5(OC1B/XCK1/MOSI)
Other:
- moved on the sheet: LED1, R21

Commit message: Added the temperature sensors
Also changed a lot of connections and PCB traces.
Parts:
- removed PDI_CONNECTOR: (no value), SparkFun-Connectors:CONN_03X2SHROUD
- added C10, C8: (no value), adafruit:C-USC0805
- added PDI: (no value), pinhead:PINHD-2X3
- added TEMP_1, TEMP_2, TEMP_3: JST-PH_3-PIN_HEADER, SRG:JST-PH_3-PIN_HEADER
- renumbered J6 to RASPBERRY, JP1 to JUMPER
Connections:
- removed net GND_RASPI: RASPBERRY.2
- removed net VCC_RASPI: RASPBERRY.6
- new net TEMP_1: TEMP_1.2, U$1.PF3(OC0D/TXD0)
- new net TEMP_2: TEMP_2.2, U$1.PF4
- new net TEMP_3: TEMP_3.2, U$1.PF5
- net DATA_RASPI: now also RASPBERRY.1; no longer RASPBERRY.5
- net GND: now also C10.2, C8.2, PDI.6, RASPBERRY.2, TEMP_1.3, TEMP_2.3, TEMP_3.3; no longer PDI_CONNECTOR.6
- net PDI_DATA: now also PDI.1; no longer PDI_CONNECTOR.1
- net RESET_PDI_CLK: now also PDI.5; no longer PDI_CONNECTOR.5
- net RES_RASPI: now also RASPBERRY.4; no longer RASPBERRY.1
- net S0: now also U$1.PC7(OC0DH/CKOUT/EVO/TXD1/SCK); no longer U$1.PC6(OC0DL/RXD1/MISO)
- net S1: now also U$1.PC6(OC0DL/RXD1/MISO); no longer U$1.PC7(OC0DH/CKOUT/EVO/TXD1/SCK)
- net TX_ATXMEGA: now also RASPBERRY.5; no longer RASPBERRY.4
- net VCC: now also C10.1, C8.1, PDI.2, RASPBERRY.6, TEMP_1.1, TEMP_2.1, TEMP_3.1; no longer PDI_CONNECTOR.2

Commit message: Added the hardware that makes the TTL line of a higher voltage.
Parts:
- removed C26: (no value), adafruit:CPOL-US175TMP-0810
- added C23: 22uF, adafruit:CPOL-US153CLV-0505
- added FAN_1, FAN_2: JST-PH_2-PIN_HEADER, SRG:JST-PH_2-PIN_HEADER
- added Q11, Q12: BSS138, SparkFun:MOSFET-NCHANNELSMD
- added R23, R24, R25: 4K7, SparkFun:RESISTOR0603-RES
- added R26, R27, R28, R29: 10K, SparkFun:RESISTOR0603-RES
- C1: value (none) -> 220uF
- C10, C11, C12, C13, C14, C15, C16, C17, C18, C19, C20, C21, C22, C3, C6, C7, C8, C9: value (none) -> 100nF
- C2: value (none) -> 220pF
- C4, C5: value (none) -> 22uF
- R21, R22: value 10K -> 330
- renumbered MOTOR_CONTROL_DEMULTIPLEXER to U4
Connections:
- net ATXMEGA_TRIGGER_1 renamed ULTRA_TRIGGER_1
- net ATXMEGA_TRIGGER_2 renamed ULTRA_TRIGGER_2
- new net FAN_1_CONTROL: FAN_1.2, U$1.PC1(OC0B/AC0AH/XCK0/SCL)
- new net FAN_2_CONTROL: FAN_2.2, U$1.PC0(OC0A/OC0AL/SDA)
- new net RX_RASPI: Q12.D, R29.2, RASPBERRY.5
- new net TX_RASPI: Q11.S, R26.2, RASPBERRY.3
- net +12V: now also C23.+, Q11.G, R26.1, R29.1; no longer C26.+
- net GND: now also C23.-, FAN_1.1, FAN_2.1, IR_1.2, IR_2.2, IR_3.2, IR_4.2, IR_5.2, IR_6.2, IR_7.2, IR_8.2; no longer C26.-, IR_1.1, IR_2.1, IR_3.1, IR_4.1, IR_5.1, IR_6.1, IR_7.1, IR_8.1
- net IR_1: now also IR_1.1; no longer IR_1.2
- net IR_2: now also IR_2.1; no longer IR_2.2
- net IR_3: now also IR_3.1; no longer IR_3.2
- net IR_4: now also IR_4.1; no longer IR_4.2
- net IR_5: now also IR_5.1; no longer IR_5.2
- net IR_6: now also IR_6.1; no longer IR_6.2
- net IR_7: now also IR_7.1; no longer IR_7.2
- net IR_8: now also IR_8.1; no longer IR_8.2
- net LED_1: now also U$1.PD4(OC1A/SS); no longer U$1.PD3(OX0D/TXD0)
- net LED_2: now also U$1.PD5(OC1B/XCK1/MOSI); no longer U$1.PD4(OC1A/SS)
- net MOTOR_CONTROL: now also U$1.PD3(OX0D/TXD0)
- net RX_ATXMEGA: now also Q11.D, R27.2; no longer RASPBERRY.3
- net TEMP_1: now also R23.2
- net TEMP_2: now also R24.2
- net TEMP_3: now also R25.2
- net TX_ATXMEGA: now also Q12.S, R28.2; no longer RASPBERRY.5
- net VCC: now also Q12.G, R23.1, R24.1, R25.1, R27.1, R28.1

Commit message: The version that is ordered at Eurocircuits.
The full version of the microcontroller PCB, revision 1.
Parts:
- J2, J3, J4: value RJ45-TRAFO -> 0446200002; device con-amphenol-rj45-ld:RJ45-TRAFO -> con-molex:0446200002
Connections:
- net GND: now also J2.1, J2.8, J2.S1, J2.S2, J3.1, J3.8, J3.S1, J3.S2, J4.1, J4.8, J4.S1, J4.S2; no longer J2.GND, J2.GND1, J2.GND2, J2.TX+, J3.GND, J3.GND1, J3.GND2, J3.TX+, J4.GND, J4.GND1, J4.GND2, J4.TX+
- net TRIGGER_1: now also J4.4; no longer J4.RX0
- net TRIGGER_2: now also J4.5; no longer J4.RX+
- net ULTRA1: now also J2.2; no longer J2.NC1
- net ULTRA10: now also J4.6; no longer J4.TX0
- net ULTRA11: now also J3.2; no longer J3.NC1
- net ULTRA12: now also J3.3; no longer J3.RX-
- net ULTRA13: now also J3.4; no longer J3.RX0
- net ULTRA14: now also J3.5; no longer J3.RX+
- net ULTRA15: now also J3.6; no longer J3.TX-
- net ULTRA16: now also J3.7; no longer J3.TX0
- net ULTRA2: now also J2.3; no longer J2.RX-
- net ULTRA3: now also J2.4; no longer J2.RX0
- net ULTRA4: now also J2.5; no longer J2.RX+
- net ULTRA5: now also J2.6; no longer J2.TX-
- net ULTRA6: now also J2.7; no longer J2.TX0
- net ULTRA7: now also J4.2; no longer J4.NC1
- net ULTRA8: now also J4.3; no longer J4.RX-
- net ULTRA9: now also J4.7; no longer J4.TX-
