File: RaspberryPi/Hardware/Raspberry Pi PCB/Raspberry Pi PCB.brd (EAGLE design)
At the start: 55 x 70 mm, 59 parts, among them Q11 BSS138, Q12 BSS138, Q2 BSS138

Commit message: Finished the Raspberry Pi PCB
Everything should be there now.
Parts:
- removed NFC: (no value), pinhead:2X05
- added C11, C12: 100nF, SparkFun-Capacitors:0805
- added GPIO4: (no value), pinhead:1X01
- added NFC_I2C: (no value), pinhead:2X03
- added NFC_SPI: (no value), pinhead:2X05
- added SELECT: (no value), jumper:SJ_2
Connections:
- removed net GP24: JP2.18
- removed net GP25: JP2.22
- removed net SCL: JP2.5
- removed net SDA: JP2.3
- new net JUMPER: JP2.22, SELECT.2
- new net NFC_SCL: JP2.5, NFC_I2C.2
- new net NFC_SDA: JP2.3, NFC_I2C.3
- net 3.3V: now also C11.1, C12.1, NFC_I2C.4, NFC_SPI.3, SELECT.1; no longer NFC.3
- net GND: now also C11.2, C12.2, NFC_I2C.5, NFC_SPI.1, NFC_SPI.2, SELECT.3; no longer NFC.1, NFC.2
- net GP4: now also GPIO4.1
- net IRQ: now also JP2.18, NFC_I2C.1, NFC_SPI.8; no longer NFC.8
- net RSTOUT_N: now also NFC_SPI.10; no longer NFC.10
- net RSTPD_N: now also NFC_SPI.9; no longer NFC.9
- net SPI_CS: now also NFC_SPI.7; no longer NFC.7
- net SPI_MISO: now also NFC_SPI.5; no longer NFC.5
- net SPI_MOSI: now also NFC_SPI.6; no longer NFC.6
- net SPI_SCK: now also NFC_SPI.4; no longer NFC.4
Routing:
- net IRQ: track 0.00 -> 65.6 mm
- net 3.3V: track 33.9 -> 83.6 mm, vias 11 -> 14
- net NFC_SCL: track 0.00 -> 38.2 mm
- net NFC_SDA: track 0.00 -> 32.8 mm
- net GP4: track 0.00 -> 24.1 mm
- net JUMPER: track 0.00 -> 21.8 mm, vias 0 -> 1
- net SPI_CS: track 46.6 -> 56.1 mm
- net SPI_SCK: track 40.8 -> 49.7 mm, vias 0 -> 1
- net SPI_MISO: track 37.9 -> 45.4 mm, vias 0 -> 1
- net GND: track 0.00 -> 3.80 mm, vias 0 -> 2
- net SPI_MOSI: track 47.4 -> 44.9 mm
Other:
- board text added: "4"
- board text added: "8"
