File: RaspberryPi/Hardware/Raspberry Pi PCB/Raspberry Pi PCB.brd (EAGLE design)
At the start: 55 x 70 mm, 64 parts, among them Q11 BSS138, Q12 BSS138, Q2 BSS138

Commit message: Added some values to the components.
These are handy when generating the BOM file.
Parts:
- R1: value (none) -> 10K
- R12, R14, R16, R18, R20, R22, R24, R26: value 10K -> 1K
- R6, R7: value (none) -> 330
- R8: value (none) -> 1K
Changed lines of the file:
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@@
 <drawing>
 <settings>
-<setting alwaysvectorfont="yes"/>
+<setting alwaysvectorfont="no"/>
 <setting verticaltext="up"/>
 </settings>
@@
 <attribute name="OC_NEWARK" value="unknown" x="28.1" y="24.6" size="1.778" layer="27" rot="R90" display="off"/>
 </element>
-<element name="R8" library="adafruit" library_urn="urn:adsk.eagle:library:420" package="R0805" value="" x="22.8" y="50.6" smashed="yes">
+<element name="R8" library="adafruit" library_urn="urn:adsk.eagle:library:420" package="R0805" value="1K" x="22.8" y="50.6" smashed="yes">
 <attribute name="NAME" x="23.397" y="52.657" size="0.8128" layer="25" rot="R180"/>
-<attribute name="VALUE" x="21.403" y="48.187" size="1.27" layer="27"/>
-</element>
-<element name="R7" library="adafruit" package="R0805" value="" x="22.45" y="24.3" smashed="yes" rot="R270">
+</element>
+<element name="R7" library="adafruit" package="R0805" value="330" x="22.45" y="24.3" smashed="yes" rot="R270">
 <attribute name="NAME" x="22.934" y="20.738" size="0.8128" layer="25" rot="R90"/>
-<attribute name="VALUE" x="20.164" y="25.062" size="1.27" layer="27" rot="R270"/>
-</element>
-<element name="R6" library="adafruit" package="R0805" value="" x="25.2" y="24.3" smashed="yes" rot="R270">
+</element>
+<element name="R6" library="adafruit" package="R0805" value="330" x="25.2" y="24.3" smashed="yes" rot="R270">
 <attribute name="NAME" x="27.184" y="23.438" size="0.8128" layer="25" rot="R90"/>
-<attribute name="VALUE" x="22.914" y="25.062" size="1.27" layer="27" rot="R270"/>
 </element>
 <element name="LED1" library="adafruit" library_urn="urn:adsk.eagle:library:420" package="CHIPLED_0805" value="" x="22.45" y="18.5" smashed="yes" rot="R180">
@@
 <attribute name="PROD_ID" value="CAP-11625" x="43.6" y="13.4" size="1.778" layer="27" rot="R270" display="off"/>
 </element>
-<element name="R1" library="adafruit" package="R0805" value="" x="35.6" y="32.1" smashed="yes" rot="R90">
+<element name="R1" library="adafruit" package="R0805" value="10K" x="35.6" y="32.1" smashed="yes" rot="R90">
 <attribute name="NAME" x="34.838" y="29.216" size="0.8128" layer="25"/>
-<attribute name="VALUE" x="37.886" y="31.338" size="1.27" layer="27" rot="R90"/>
 </element>
 <element name="REED" library="con-molex" library_urn="urn:adsk.eagle:library:165" package="7395-02" value="22-05-7028-02" x="49.5" y="37.6" smashed="yes" rot="R90">
@@
 </element>
 <element name="R11" library="SparkFun" package="0603-RES" value="10K" x="2.3" y="61.2" rot="R90"/>
-<element name="R12" library="SparkFun" package="0603-RES" value="10K" x="4.8" y="61.2" rot="R270"/>
+<element name="R12" library="SparkFun" package="0603-RES" value="1K" x="4.8" y="61.2" rot="R270"/>
 <element name="R13" library="SparkFun" package="0603-RES" value="10K" x="8.7" y="61.2" rot="R90"/>
-<element name="R14" library="SparkFun" package="0603-RES" value="10K" x="11.3" y="61.2" rot="R270"/>
+<element name="R14" library="SparkFun" package="0603-RES" value="1K" x="11.3" y="61.2" rot="R270"/>
 <element name="R15" library="SparkFun" package="0603-RES" value="10K" x="15.4" y="61.2" rot="R90"/>
-<element name="R16" library="SparkFun" package="0603-RES" value="10K" x="17.9" y="61.2" rot="R270"/>
+<element name="R16" library="SparkFun" package="0603-RES" value="1K" x="17.9" y="61.2" rot="R270"/>
 <element name="R17" library="SparkFun" package="0603-RES" value="10K" x="22.2" y="61.2" rot="R90"/>
-<element name="R18" library="SparkFun" package="0603-RES" value="10K" x="24.8" y="61.2" rot="R270"/>
+<element name="R18" library="SparkFun" package="0603-RES" value="1K" x="24.8" y="61.2" rot="R270"/>
 <element name="R19" library="SparkFun" package="0603-RES" value="10K" x="29.4" y="61.2" rot="R90"/>
-<element name="R20" library="SparkFun" package="0603-RES" value="10K" x="32" y="61.2" rot="R270"/>
+<element name="R20" library="SparkFun" package="0603-RES" value="1K" x="32" y="61.2" rot="R270"/>
 <element name="R21" library="SparkFun" package="0603-RES" value="10K" x="36.1" y="61.2" rot="R90"/>
-<element name="R22" library="SparkFun" package="0603-RES" value="10K" x="38.7" y="61.2" rot="R270"/>
+<element name="R22" library="SparkFun" package="0603-RES" value="1K" x="38.7" y="61.2" rot="R270"/>
 <element name="R23" library="SparkFun" package="0603-RES" value="10K" x="42.9" y="61.2" rot="R90"/>
-<element name="R24" library="SparkFun" package="0603-RES" value="10K" x="45.5" y="61.2" rot="R270"/>
+<element name="R24" library="SparkFun" package="0603-RES" value="1K" x="45.5" y="61.2" rot="R270"/>
 <element name="R25" library="SparkFun" package="0603-RES" value="10K" x="49.7" y="61.2" rot="R90"/>
-<element name="R26" library="SparkFun" package="0603-RES" value="10K" x="52.3" y="61.2" rot="R270"/>
+<element name="R26" library="SparkFun" package="0603-RES" value="1K" x="52.3" y="61.2" rot="R270"/>
 <element name="SELECT" library="jumper" library_urn="urn:adsk.eagle:library:252" package="SJ_2" package3d_urn="urn:adsk.eagle:package:15474/1" value="" x="16.75" y="29.5" smashed="yes" rot="R180">
 <attribute name="NAME" x="15.237" y="30.67" size="0.6096" layer="25" ratio="10"/>
