File: RaspberryPi/Hardware/Raspberry Pi PCB/Raspberry Pi PCB.sch (EAGLE design)
At the start: 59 parts, among them Q11 BSS138, Q12 BSS138, Q2 BSS138

Commit message: Finished the Raspberry Pi PCB
Everything should be there now.
Parts:
- removed NFC: (no value), pinhead:PINHD-2X5
- added C11, C12: 100nF, SparkFun-Capacitors:1.0UF-0805-25V-(+80/-20%)
- added GPIO4: (no value), pinhead:PINHD-1X1
- added NFC_I2C: (no value), pinhead:PINHD-2X3
- added NFC_SPI: (no value), pinhead:PINHD-2X5
- added SELECT: (no value), jumper:SJ2W
Connections:
- removed net GP24: JP2.GP24
- removed net GP25: JP2.GP25
- removed net SCL: JP2.SCL
- removed net SDA: JP2.SDA
- new net JUMPER: JP2.GP25, SELECT.2
- new net NFC_SCL: JP2.SCL, NFC_I2C.2
- new net NFC_SDA: JP2.SDA, NFC_I2C.3
- net 3.3V: now also C11.1, C12.1, NFC_I2C.4, NFC_SPI.3, SELECT.1; no longer NFC.3
- net GND: now also C11.2, C12.2, NFC_I2C.5, NFC_SPI.1, NFC_SPI.2, SELECT.3; no longer NFC.1, NFC.2
- net GP4: now also GPIO4.1
- net IRQ: now also JP2.GP24, NFC_I2C.1, NFC_SPI.8; no longer NFC.8
- net RSTOUT_N: now also NFC_SPI.10; no longer NFC.10
- net RSTPD_N: now also NFC_SPI.9; no longer NFC.9
- net SPI_CS: now also NFC_SPI.7; no longer NFC.7
- net SPI_MISO: now also NFC_SPI.5; no longer NFC.5
- net SPI_MOSI: now also NFC_SPI.6; no longer NFC.6
- net SPI_SCK: now also NFC_SPI.4; no longer NFC.4
Other:
- note added: "Machine size selection"
- note added: "The Raspberry Pi GPIO is only 3.3V, this needs to be 5V."
- note removed: "Between these terminals the reed switch is connected"
- note removed: "kolommen selectie: 4 of 8 stuks"
- moved on the sheet: BUTTON1-1, BUTTON1-2, BUTTON2-1, BUTTON2-2, BUTTON3-1, BUTTON3-2, BUTTON4-1, BUTTON4-2, BUTTON5-1, BUTTON5-2, BUTTON6-1, BUTTON6-2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

Commit message: Added some values to the components.
These are handy when generating the BOM file.
Parts:
- R1: value (none) -> 10K
- R12, R14, R16, R18, R20, R22, R24, R26: value 10K -> 1K
- R6, R7: value (none) -> 330
- R8: value (none) -> 1K
Changed lines of the file:
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@@
 <part name="GND21" library="SparkFun" deviceset="GND" device=""/>
 <part name="GND22" library="SparkFun" deviceset="GND" device=""/>
-<part name="R8" library="adafruit" library_urn="urn:adsk.eagle:library:420" deviceset="R-US_" device="R0805"/>
-<part name="R7" library="adafruit" deviceset="R-US_" device="R0805"/>
-<part name="R6" library="adafruit" deviceset="R-US_" device="R0805"/>
+<part name="R8" library="adafruit" library_urn="urn:adsk.eagle:library:420" deviceset="R-US_" device="R0805" value="1K"/>
+<part name="R7" library="adafruit" deviceset="R-US_" device="R0805" value="330"/>
+<part name="R6" library="adafruit" deviceset="R-US_" device="R0805" value="330"/>
 <part name="GND23" library="SparkFun" deviceset="GND" device=""/>
 <part name="GND24" library="SparkFun" deviceset="GND" device=""/>
@@
 <part name="C7" library="SparkFun-Capacitors" library_urn="urn:adsk.eagle:library:510" deviceset="1.0UF" device="-0805-25V-(+80/-20%)" package3d_urn="urn:adsk.eagle:package:37429/1" value="100nF"/>
 <part name="SUPPLY3" library="SparkFun-Aesthetics" deviceset="3.3V" device=""/>
-<part name="R1" library="adafruit" deviceset="R-US_" device="R0805"/>
+<part name="R1" library="adafruit" deviceset="R-US_" device="R0805" value="10K"/>
 <part name="REED" library="con-molex" library_urn="urn:adsk.eagle:library:165" deviceset="22-?-02" device="05-7028"/>
 <part name="GND15" library="SparkFun" deviceset="GND" device=""/>
@@
 <part name="SUPPLY5" library="SparkFun-Aesthetics" deviceset="3.3V" device=""/>
 <part name="R11" library="SparkFun" deviceset="RESISTOR" device="0603-RES" value="10K"/>
-<part name="R12" library="SparkFun" deviceset="RESISTOR" device="0603-RES" value="10K"/>
+<part name="R12" library="SparkFun" deviceset="RESISTOR" device="0603-RES" value="1K"/>
 <part name="SUPPLY6" library="SparkFun-Aesthetics" deviceset="3.3V" device=""/>
 <part name="R13" library="SparkFun" deviceset="RESISTOR" device="0603-RES" value="10K"/>
-<part name="R14" library="SparkFun" deviceset="RESISTOR" device="0603-RES" value="10K"/>
+<part name="R14" library="SparkFun" deviceset="RESISTOR" device="0603-RES" value="1K"/>
 <part name="SUPPLY10" library="SparkFun-Aesthetics" deviceset="3.3V" device=""/>
 <part name="R15" library="SparkFun" deviceset="RESISTOR" device="0603-RES" value="10K"/>
-<part name="R16" library="SparkFun" deviceset="RESISTOR" device="0603-RES" value="10K"/>
+<part name="R16" library="SparkFun" deviceset="RESISTOR" device="0603-RES" value="1K"/>
 <part name="SUPPLY11" library="SparkFun-Aesthetics" deviceset="3.3V" device=""/>
 <part name="R17" library="SparkFun" deviceset="RESISTOR" device="0603-RES" value="10K"/>
-<part name="R18" library="SparkFun" deviceset="RESISTOR" device="0603-RES" value="10K"/>
+<part name="R18" library="SparkFun" deviceset="RESISTOR" device="0603-RES" value="1K"/>
 <part name="SUPPLY12" library="SparkFun-Aesthetics" deviceset="3.3V" device=""/>
 <part name="R19" library="SparkFun" deviceset="RESISTOR" device="0603-RES" value="10K"/>
-<part name="R20" library="SparkFun" deviceset="RESISTOR" device="0603-RES" value="10K"/>
+<part name="R20" library="SparkFun" deviceset="RESISTOR" device="0603-RES" value="1K"/>
 <part name="SUPPLY15" library="SparkFun-Aesthetics" deviceset="3.3V" device=""/>
 <part name="R21" library="SparkFun" deviceset="RESISTOR" device="0603-RES" value="10K"/>
-<part name="R22" library="SparkFun" deviceset="RESISTOR" device="0603-RES" value="10K"/>
+<part name="R22" library="SparkFun" deviceset="RESISTOR" device="0603-RES" value="1K"/>
 <part name="SUPPLY16" library="SparkFun-Aesthetics" deviceset="3.3V" device=""/>
 <part name="R23" library="SparkFun" deviceset="RESISTOR" device="0603-RES" value="10K"/>
-<part name="R24" library="SparkFun" deviceset="RESISTOR" device="0603-RES" value="10K"/>
+<part name="R24" library="SparkFun" deviceset="RESISTOR" device="0603-RES" value="1K"/>
 <part name="SUPPLY17" library="SparkFun-Aesthetics" deviceset="3.3V" device=""/>
 <part name="R25" library="SparkFun" deviceset="RESISTOR" device="0603-RES" value="10K"/>
-<part name="R26" library="SparkFun" deviceset="RESISTOR" device="0603-RES" value="10K"/>
+<part name="R26" library="SparkFun" deviceset="RESISTOR" device="0603-RES" value="1K"/>
 <part name="SELECT" library="jumper" library_urn="urn:adsk.eagle:library:252" deviceset="SJ2W" device="" package3d_urn="urn:adsk.eagle:package:15474/1"/>
 <part name="GND33" library="SparkFun" deviceset="GND" device=""/>
